Commit message: camera attached on UR5

File: urdf/ur5_with_camera.urdf.xacro (robot description, xacro)
@@ -1,6 +1,6 @@
 <?xml version="1.0"?>
 <robot xmlns:xacro="http://ros.org/wiki/xacro">
-  <xacro:include filename="$(find ur_description)/urdf/ur.transmission.xacro" />
-  <xacro:include filename="$(find ur_description)/urdf/ur.gazebo.xacro" />
+  <xacro:include filename="$(find ur5_with_hand_gazebo)/urdf/ur.transmission.xacro" />
+  <xacro:include filename="$(find ur5_with_hand_gazebo)/urdf/ur5_with_camera.gazebo.xacro" />
   <!-- Inertia parameters -->
   <xacro:property name="base_mass" value="4.0" />  <!-- This mass might be incorrect -->
@@ -295,5 +295,5 @@
 		<link name="camera_link">
 			<collision>
-				<origin xyz="0 0 0" rpy="0 0 0"/>
+				<origin xyz="0 0 0.1" rpy="0 0 0"/>
 				<geometry>
 			<box size="${camera_link} ${camera_link} ${camera_link}"/>
@@ -301,4 +301,5 @@
 			</collision>
 			<visual>
+				<transparency>1</transparency>
 				<origin xyz="0 0 0" rpy="0 0 0"/>
 				<geometry>
@@ -316,5 +317,5 @@
       <parent link="${prefix}wrist_3_link" />
       <child link = "camera_link" />
-      <origin xyz="${wrist_3_length / -2.0} ${wrist_3_length} 0.0" rpy="0.0 0.0 ${pi/2.0}" />
+      <origin xyz="0.0 ${wrist_3_length} ${wrist_3_length / 2.0}" rpy="0.0 0.0 ${pi/2.0}" />
     </joint>
     <xacro:ur_arm_transmission prefix="${prefix}" />
