Commit message: tool pose is sent correctly in this way but cannot subscribe \tool0

File: urdf/ur.gazebo.xacro (robot description, xacro)
@@ -26,6 +26,6 @@
 			<plugin name="ground_truth" filename="libgazebo_ros_p3d.so">
 				<frameName>map</frameName>
-				<bodyName>${prefix}ee_link</bodyName>
-				<topicName>odom_ee_link</topicName>
+				<bodyName>${prefix}tool0</bodyName>
+				<topicName>odom_tool0</topicName>
 				<updateRate>30.0</updateRate>
 			</plugin>

File: urdf/ur5.urdf.xacro (robot description, xacro)
@@ -336,4 +336,5 @@
     <joint name="${prefix}wrist_3_link-tool0_fixed_joint" type="fixed">
       <origin xyz="0 ${wrist_3_length} 0" rpy="${pi/-2.0} 0 0"/>
+      <!--<origin xyz="0 0 0" rpy="0 0 0"/>  To trick Gazebo/Moveit pose planner. Find a better way later-->
       <parent link="${prefix}wrist_3_link"/>
       <child link="${prefix}tool0"/>
