Commit message: to load just wrist available urdf -- careful on world link

File: urdf/ur5_robot.urdf.xacro (robot description, xacro)
@@ -5,7 +5,8 @@
   <xacro:include filename="$(find ur5_with_hand_gazebo)/urdf/common.gazebo.xacro" />
   <!-- ur5 -->
-  <xacro:include filename="$(find ur5_with_hand_gazebo)/urdf/ur5.urdf.xacro" />
+	<xacro:include filename="$(find ur5_with_hand_gazebo)/urdf/ur5-fhdesc-wristonly.urdf"/>
+  <!--<xacro:include filename="$(find ur5_with_hand_gazebo)/urdf/ur5.urdf.xacro" />-->
   <!--<xacro:include filename="$(find ur5_with_hand_gazebo)/urdf/ur5_with_camera.urdf.xacro" />-->
-  <!-- arm -->
+  <!-- arm
   <xacro:ur5_robot prefix="" joint_limited="false"/>
   <link name="world" />
@@ -14,4 +15,4 @@
     <child link = "base_link" />
     <origin xyz="0.0 0.0 0.0" rpy="0.0 0.0 0.0" />
-  </joint>
+  </joint>-->
 </robot>
