Commit message: wrist controller seperated - There is conflict

File: urdf/ur5-fhdesc-wristonly.urdf (robot description, URDF)
Before this commit: robot ur5, 11 links, 10 joints
Joints:
- joint elbow_joint: type revolute -> fixed
- joint world_joint: origin xyz=0.0 -1.0 1.0 rpy=0.0 0.0 0.0 -> xyz=0.0 0.0 0.0 rpy=0.0 0.0 0.0
- joint wrist_1_joint: origin xyz=0.0 0.0 0.5723 rpy=0.0 3.1415 0.0 -> xyz=0.0 0.0 0.5723 rpy=0.0 0.0 0.0

File: urdf/ur5_robot.urdf.xacro (robot description, xacro)
@@ -5,8 +5,8 @@
   <xacro:include filename="$(find ur5_with_hand_gazebo)/urdf/common.gazebo.xacro" />
   <!-- ur5 -->
-	<xacro:include filename="$(find ur5_with_hand_gazebo)/urdf/ur5-fhdesc-wristonly.urdf"/>
-  <!--<xacro:include filename="$(find ur5_with_hand_gazebo)/urdf/ur5.urdf.xacro" />-->
+	<!--<xacro:include filename="$(find ur5_with_hand_gazebo)/urdf/ur5-fhdesc-wristonly.urdf"/>-->
+  <xacro:include filename="$(find ur5_with_hand_gazebo)/urdf/ur5.urdf.xacro" />
   <!--<xacro:include filename="$(find ur5_with_hand_gazebo)/urdf/ur5_with_camera.urdf.xacro" />-->
-  <!-- arm
+  <!-- arm -->
   <xacro:ur5_robot prefix="" joint_limited="false"/>
   <link name="world" />
@@ -15,4 +15,4 @@
     <child link = "base_link" />
     <origin xyz="0.0 0.0 0.0" rpy="0.0 0.0 0.0" />
-  </joint>-->
+  </joint>
 </robot>
