Commit message: UR5 initial pose updated

File: urdf/ur5.urdf.xacro (robot description, xacro)
@@ -95,5 +95,5 @@
       <parent link="${prefix}base_link" />
       <child link = "${prefix}shoulder_link" />
-      <origin xyz="0.0 0.0 ${shoulder_height}" rpy="0.0 0.0 0.0" />
+      <origin xyz="0.0 0.0 ${shoulder_height}" rpy="0.0 ${pi / -2.0} 0.0" />
       <axis xyz="0 0 1" />
       <xacro:unless value="${joint_limited}">
@@ -188,5 +188,5 @@
       <parent link="${prefix}forearm_link" />
       <child link = "${prefix}wrist_1_link" />
-      <origin xyz="0.0 0.0 ${forearm_length}" rpy="0.0 ${pi / 2.0} 0.0" />
+      <origin xyz="0.0 0.0 ${forearm_length}" rpy="0.0 0.0 0.0" />
       <axis xyz="0 1 0" />
       <xacro:unless value="${joint_limited}">

Commit message: no camera, ur5_gizem_moveit_config works with that model

File: urdf/ur5.urdf.xacro (robot description, xacro)
@@ -2,5 +2,5 @@
 <robot xmlns:xacro="http://ros.org/wiki/xacro">
   <xacro:include filename="$(find ur_description)/urdf/ur.transmission.xacro" />
-  <xacro:include filename="$(find ur_description)/urdf/ur.gazebo.xacro" />
+  <xacro:include filename="$(find ur5_with_hand_gazebo)/urdf/ur5_with_camera.gazebo.xacro" />
   <!-- Inertia parameters -->
   <xacro:property name="base_mass" value="4.0" />  <!-- This mass might be incorrect -->
@@ -95,5 +95,5 @@
       <parent link="${prefix}base_link" />
       <child link = "${prefix}shoulder_link" />
-      <origin xyz="0.0 0.0 ${shoulder_height}" rpy="0.0 ${pi / -2.0} 0.0" />
+      <origin xyz="0.0 0.0 ${shoulder_height}" rpy="0.0 0.0 0.0" />
       <axis xyz="0 0 1" />
       <xacro:unless value="${joint_limited}">
@@ -188,5 +188,5 @@
       <parent link="${prefix}forearm_link" />
       <child link = "${prefix}wrist_1_link" />
-      <origin xyz="0.0 0.0 ${forearm_length}" rpy="0.0 0.0 0.0" />
+      <origin xyz="0.0 0.0 ${forearm_length}" rpy="0.0 ${pi / 2.0} 0.0" />
       <axis xyz="0 1 0" />
       <xacro:unless value="${joint_limited}">
@@ -291,4 +291,32 @@
       </collision>
     </link>
+        <!-- Camera -->
+    <xacro:property name="camera_link" value="0.05" /> <!-- Size of square 'camera' box -->
+		<!--<link name="camera_link">
+			<collision>
+				<origin xyz="0 0 0.1" rpy="0 0 0"/>
+				<geometry>
+			<box size="${camera_link} ${camera_link} ${camera_link}"/>
+				</geometry>
+			</collision>
+			<visual>
+				<transparency>1</transparency>
+				<origin xyz="0 0 0" rpy="0 0 0"/>
+				<geometry>
+			<box size="${camera_link} ${camera_link} ${camera_link}"/>
+				</geometry>
+				<material name="red"/>
+			</visual>
+			<inertial>
+				<mass value="0" />
+				<origin xyz="0 0 0" rpy="0 0 0"/>
+				<inertia ixx="1e-6" ixy="0" ixz="0" iyy="1e-6" iyz="0" izz="1e-6" />
+			</inertial>
+		</link>
+		<joint name="camera_fixed_joint" type="fixed">
+      <parent link="${prefix}wrist_3_link" />
+      <child link = "camera_link" />
+      <origin xyz="0.0 ${wrist_3_length} ${wrist_3_length / 2.0}" rpy="0.0 0.0 ${pi/2.0}" />
+    </joint>	-->
     <xacro:ur_arm_transmission prefix="${prefix}" />
     <xacro:ur_arm_gazebo prefix="${prefix}" />

File: urdf/ur5_robot.urdf.xacro (robot description, xacro)
@@ -5,6 +5,6 @@
   <xacro:include filename="$(find ur5_with_hand_gazebo)/urdf/common.gazebo.xacro" />
   <!-- ur5 -->
-  <!--<xacro:include filename="$(find ur5_with_hand_gazebo)/urdf/ur5.urdf.xacro" />-->
-  <xacro:include filename="$(find ur5_with_hand_gazebo)/urdf/ur5_with_camera.urdf.xacro" />
+  <xacro:include filename="$(find ur5_with_hand_gazebo)/urdf/ur5.urdf.xacro" />
+  <!--<xacro:include filename="$(find ur5_with_hand_gazebo)/urdf/ur5_with_camera.urdf.xacro" />-->
   <!-- arm -->
   <xacro:ur5_robot prefix="" joint_limited="false"/>

Commit message: I wanna cry. It works as before again. Thanks universe.

File: urdf/ur5.urdf.xacro (robot description, xacro)
@@ -1,5 +1,5 @@
 <?xml version="1.0"?>
 <robot xmlns:xacro="http://ros.org/wiki/xacro">
-  <xacro:include filename="$(find ur_description)/urdf/ur.transmission.xacro" />
+  <xacro:include filename="$(find ur5_with_hand_gazebo)/urdf/ur.transmission.xacro" />
   <xacro:include filename="$(find ur5_with_hand_gazebo)/urdf/ur.gazebo.xacro" />
   <!-- Inertia parameters -->
@@ -291,7 +291,7 @@
       </collision>
     </link>
-        <!-- Camera -->
-    <xacro:property name="camera_link" value="0.05" /> <!-- Size of square 'camera' box -->
-		<!--<link name="camera_link">
+    <!-- Camera
+    <xacro:property name="camera_link" value="0.05" />
+		<link name="camera_link">
 			<collision>
 				<origin xyz="0 0 0.1" rpy="0 0 0"/>
@@ -309,5 +309,5 @@
 			</visual>
 			<inertial>
-				<mass value="0" />
+				<mass value="1e-5" />
 				<origin xyz="0 0 0" rpy="0 0 0"/>
 				<inertia ixx="1e-6" ixy="0" ixz="0" iyy="1e-6" iyz="0" izz="1e-6" />
@@ -336,5 +336,5 @@
     <joint name="${prefix}wrist_3_link-tool0_fixed_joint" type="fixed">
       <origin xyz="0 ${wrist_3_length} 0" rpy="${pi/-2.0} 0 0"/>
-      <!--<origin xyz="0 0 0" rpy="0 0 0"/>  To trick Gazebo/Moveit pose planner. Find a better way later-->
+<!--<origin xyz="0 0 0" rpy="0 0 0"/>  To trick Gazebo/Moveit pose planner. Find a better way later-->
       <parent link="${prefix}wrist_3_link"/>
       <child link="${prefix}tool0"/>

File: urdf/ur5_robot.urdf.xacro (robot description, xacro)
@@ -6,6 +6,6 @@
   <!-- ur5 -->
 	<!--<xacro:include filename="$(find ur_e_description)/urdf/ur5e_robot.urdf.xacro" />-->
-  <!--<xacro:include filename="$(find ur5_with_hand_gazebo)/urdf/ur5.urdf.xacro" />-->
-  <xacro:include filename="$(find ur5_with_hand_gazebo)/urdf/ur5_with_camera.urdf.xacro" />
+  <xacro:include filename="$(find ur5_with_hand_gazebo)/urdf/ur5.urdf.xacro" />
+  <!--<xacro:include filename="$(find ur5_with_hand_gazebo)/urdf/ur5_with_camera.urdf.xacro" />-->
   <!-- arm -->
   <xacro:ur5_robot prefix="" joint_limited="false"/>

File: urdf/ur5_with_camera.urdf.xacro (robot description, xacro)
@@ -95,5 +95,5 @@
       <parent link="${prefix}base_link" />
       <child link = "${prefix}shoulder_link" />
-      <origin xyz="0.0 0.0 ${shoulder_height}" rpy="0.0 ${pi / -2.0} 0.0" />
+      <origin xyz="0.0 0.0 ${shoulder_height}" rpy="0.0 0.0 0.0" />
       <axis xyz="0 0 1" />
       <xacro:unless value="${joint_limited}">
@@ -188,5 +188,5 @@
       <parent link="${prefix}forearm_link" />
       <child link = "${prefix}wrist_1_link" />
-      <origin xyz="0.0 0.0 ${forearm_length}" rpy="0.0 0.0 0.0" />
+      <origin xyz="0.0 0.0 ${forearm_length}" rpy="0.0 ${pi / 2.0} 0.0" />
       <axis xyz="0 1 0" />
       <xacro:unless value="${joint_limited}">
@@ -318,5 +318,5 @@
       <child link = "camera_link" />
       <origin xyz="0.0 ${wrist_3_length} ${wrist_3_length / 2.0}" rpy="0.0 0.0 ${pi/2.0}" />
-    </joint>
+    </joint>	-->
     <xacro:ur_arm_transmission prefix="${prefix}" />
     <xacro:ur_arm_gazebo prefix="${prefix}" />
@@ -336,4 +336,5 @@
     <joint name="${prefix}wrist_3_link-tool0_fixed_joint" type="fixed">
       <origin xyz="0 ${wrist_3_length} 0" rpy="${pi/-2.0} 0 0"/>
+<!--<origin xyz="0 0 0" rpy="0 0 0"/>  To trick Gazebo/Moveit pose planner. Find a better way later-->
       <parent link="${prefix}wrist_3_link"/>
       <child link="${prefix}tool0"/>
